Commit message: ikfast

File: ws_ros2_hanwha/src/hcr3a/urdf/hcr3a.urdf (robot description, URDF)
Before this commit: robot hcr3a, 18 links, 17 joints
Links:
- removed link base
- removed link camera_depth_optical_frame
- link base_link: geometry collision mesh filename=file:///home/mmazur/Prace/ImieNN/MecHaRo-Lab_HCR3a/ws_ros2_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; visual mesh filename=file:///home/mmazur/Prace/ImieNN/MecHaRo-Lab_HCR3a/ws_ros2_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
- link camera_Link: geometry collision mesh filename=file:///home/mmazur/Prace/ImieNN/MecHaRo-Lab_HCR3a/ws_ros2_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; visual mesh filename=file:///home/mmazur/Prace/ImieNN/MecHaRo-Lab_HCR3a/ws_ros2_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
- link camera_link: geometry collision box size=0.02005 0.099 0.023; visual mesh filename=file:///opt/ros/jazzy/share/realsense2_description/meshes/d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
- link effector_Link: geometry collision mesh filename=file:///home/mmazur/Prace/ImieNN/MecHaRo-Lab_HCR3a/ws_ros2_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; visual mesh filename=file:///home/mmazur/Prace/ImieNN/MecHaRo-Lab_HCR3a/ws_ros2_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
- link finger1_Link: geometry collision mesh filename=file:///home/mmazur/Prace/ImieNN/MecHaRo-Lab_HCR3a/ws_ros2_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; visual mesh filename=file:///home/mmazur/Prace/ImieNN/MecHaRo-Lab_HCR3a/ws_ros2_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
- link finger2_Link: geometry collision mesh filename=file:///home/mmazur/Prace/ImieNN/MecHaRo-Lab_HCR3a/ws_ros2_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; visual mesh filename=file:///home/mmazur/Prace/ImieNN/MecHaRo-Lab_HCR3a/ws_ros2_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
- link forcesensor_Link: geometry collision mesh filename=file:///home/mmazur/Prace/ImieNN/MecHaRo-Lab_HCR3a/ws_ros2_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; visual mesh filename=file:///home/mmazur/Prace/ImieNN/MecHaRo-Lab_HCR3a/ws_ros2_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
- link link_1: geometry collision mesh filename=file:///home/mmazur/Prace/ImieNN/MecHaRo-Lab_HCR3a/ws_ros2_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; visual mesh filename=file:///home/mmazur/Prace/ImieNN/MecHaRo-Lab_HCR3a/ws_ros2_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
- link link_2: geometry collision mesh filename=file:///home/mmazur/Prace/ImieNN/MecHaRo-Lab_HCR3a/ws_ros2_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; visual mesh filename=file:///home/mmazur/Prace/ImieNN/MecHaRo-Lab_HCR3a/ws_ros2_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
- link link_3: geometry collision mesh filename=file:///home/mmazur/Prace/ImieNN/MecHaRo-Lab_HCR3a/ws_ros2_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; visual mesh filename=file:///home/mmazur/Prace/ImieNN/MecHaRo-Lab_HCR3a/ws_ros2_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
- link link_4: geometry collision mesh filename=file:///home/mmazur/Prace/ImieNN/MecHaRo-Lab_HCR3a/ws_ros2_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; visual mesh filename=file:///home/mmazur/Prace/ImieNN/MecHaRo-Lab_HCR3a/ws_ros2_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
- link link_5: geometry collision mesh filename=file:///home/mmazur/Prace/ImieNN/MecHaRo-Lab_HCR3a/ws_ros2_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; visual mesh filename=file:///home/mmazur/Prace/ImieNN/MecHaRo-Lab_HCR3a/ws_ros2_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
- link link_6: geometry collision mesh filename=file:///home/mmazur/Prace/ImieNN/MecHaRo-Lab_HCR3a/ws_ros2_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; visual mesh filename=file:///home/mmazur/Prace/ImieNN/MecHaRo-Lab_HCR3a/ws_ros2_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
Joints:
- removed joint base_link-base
- removed joint {prefix}camera_depth_optical_link
- joint finger1: limit lower=0 upper=0.02557 effort=0 velocity=0 -> lower=-0.1 upper=0.03 effort=150.0 velocity=1000.0
- joint finger2: limit lower=-0.02557 upper=0 effort=0 velocity=0 -> lower=-0.03 upper=0.1 effort=150.0 velocity=1000.0; mimic joint=finger1 multiplier=-1 offset=0 -> (none)
- joint forcesensor: axis 0 0 0 -> 1 0 0; limit (none) -> lower=-0.0 upper=0.0 effort=5000.0 velocity=0.01
- joint joint_1: limit lower=-6.2832 upper=6.2832 effort=0 velocity=3.1416 -> lower=-6.2832 upper=6.2832 effort=150.0 velocity=3.1416
- joint joint_2: limit lower=-6.2832 upper=6.2832 effort=0 velocity=3.1416 -> lower=-6.2832 upper=6.2832 effort=150.0 velocity=3.1416
- joint joint_3: limit lower=-2.7925 upper=2.7925 effort=0 velocity=3.1416 -> lower=-2.7925 upper=2.7925 effort=150.0 velocity=3.1416
- joint joint_4: limit lower=-6.2832 upper=6.2832 effort=0 velocity=6.2832 -> lower=-6.2832 upper=6.2832 effort=150. velocity=6.2832
- joint joint_5: limit lower=-6.2832 upper=6.2832 effort=0 velocity=6.2832 -> lower=-6.2832 upper=6.2832 effort=150.0 velocity=6.2832
- joint joint_6: limit lower=-3.146 upper=3.146 effort=0 velocity=6.2832 -> lower=-3.146 upper=3.146 effort=150.0 velocity=6.2832
