Commit message: servo fix

File: ws_ros2_hanwha/src/hcr3a/urdf/hcr3a_macro.xacro (robot description, xacro)
@@ -378,5 +378,5 @@
     <limit lower="-0.03" upper="0.1" effort="150.0" velocity="1000.0" />
     <dynamics damping="0" friction="0"/>
-    <!-- mimic joint="${prefix}finger1" multiplier="-1" offset="0" /-->
+    <mimic joint="${prefix}finger1" multiplier="-1" offset="0" />
   </joint>
     <!-- end of joint list -->
