Commit message: controller launch configs updated

File: ws_ros2_hanwha/src/hcr3a/urdf/hcr3a_macro.xacro (robot description, xacro)
@@ -4,5 +4,6 @@
   <xacro:macro name="hcr3a" params="prefix">
   <!-- link list -->
-  <link name="${prefix}base_link">
+  <link name="${prefix}base_link"/>
+  <link name="${prefix}real_base_link">
     <inertial>
       <origin xyz="7.97584139442861E-05 -0.0005270967790151 0.016153272685018" rpy="0 0 0" />
@@ -295,7 +296,12 @@
   </link>
     <!-- end of link list -->
+  <joint name="${prefix}joint_0" type="fixed">
+    <origin xyz="0 0 0.0" rpy="0 0 0" />
+    <parent link="${prefix}base_link" />
+    <child link="${prefix}real_base_link" />
+  </joint>
   <joint name="${prefix}joint_1" type="revolute">
     <origin xyz="0 0 0.03769" rpy="1.5708 0 1.5708" />
-    <parent link="${prefix}base_link" />
+    <parent link="${prefix}real_base_link" />
     <child link="${prefix}link_1" />
     <axis xyz="0 1 0"  />

Commit message: path in xacro correction

File: ws_ros2_hanwha/src/hcr3a/urdf/hcr3a_macro.xacro (robot description, xacro)
@@ -16,5 +16,5 @@
       <origin xyz="0 0 0" rpy="0 0 0" />
       <geometry>
-        <mesh filename="file://$(find hcr3a)/meshes/visual/base_link.STL" />
+        <mesh filename="package://hcr3a/meshes/visual/base_link.STL" />
       </geometry>
       <material name="">
@@ -25,5 +25,5 @@
       <origin xyz="0 0 0" rpy="0 0 0" />
       <geometry>
-        <mesh filename="file://$(find hcr3a)/meshes/visual/base_link.STL" />
+        <mesh filename="package://hcr3a/meshes/visual/base_link.STL" />
       </geometry>
     </collision>
@@ -40,5 +40,5 @@
       <origin xyz="0 0 0" rpy="0 0 0" />
       <geometry>
-        <mesh filename="file://$(find hcr3a)/meshes/visual/Link_1.STL" />
+        <mesh filename="package://hcr3a/meshes/visual/Link_1.STL" />
       </geometry>
       <material name="">
@@ -49,5 +49,5 @@
       <origin xyz="0 0 0" rpy="0 0 0" />
       <geometry>
-        <mesh filename="file://$(find hcr3a)/meshes/visual/Link_1.STL" />
+        <mesh filename="package://hcr3a/meshes/visual/Link_1.STL" />
       </geometry>
     </collision>
@@ -64,5 +64,5 @@
       <origin xyz="0 0 0" rpy="0 0 0" />
       <geometry>
-        <mesh filename="file://$(find hcr3a)/meshes/visual/Link_2.STL" />
+        <mesh filename="package://hcr3a/meshes/visual/Link_2.STL" />
       </geometry>
       <material name="">
@@ -73,5 +73,5 @@
       <origin xyz="0 0 0" rpy="0 0 0" />
       <geometry>
-        <mesh filename="file://$(find hcr3a)/meshes/visual/Link_2.STL" />
+        <mesh filename="package://hcr3a/meshes/visual/Link_2.STL" />
       </geometry>
     </collision>
@@ -88,5 +88,5 @@
       <origin xyz="0 0 0" rpy="0 0 0" />
       <geometry>
-        <mesh filename="file://$(find hcr3a)/meshes/visual/Link_3.STL" />
+        <mesh filename="package://hcr3a/meshes/visual/Link_3.STL" />
       </geometry>
       <material
@@ -98,5 +98,5 @@
       <origin xyz="0 0 0" rpy="0 0 0" />
       <geometry>
-        <mesh filename="file://$(find hcr3a)/meshes/visual/Link_3.STL" />
+        <mesh filename="package://hcr3a/meshes/visual/Link_3.STL" />
       </geometry>
     </collision>
@@ -113,5 +113,5 @@
       <origin xyz="0 0 0" rpy="0 0 0" />
       <geometry>
-        <mesh filename="file://$(find hcr3a)/meshes/visual/Link_4.STL" />
+        <mesh filename="package://hcr3a/meshes/visual/Link_4.STL" />
       </geometry>
       <material name="">
@@ -122,5 +122,5 @@
       <origin xyz="0 0 0" rpy="0 0 0" />
       <geometry>
-        <mesh filename="file://$(find hcr3a)/meshes/visual/Link_4.STL" />
+        <mesh filename="package://hcr3a/meshes/visual/Link_4.STL" />
       </geometry>
     </collision>
@@ -137,5 +137,5 @@
       <origin xyz="0 0 0" rpy="0 0 0" />
       <geometry>
-        <mesh filename="file://$(find hcr3a)/meshes/visual/Link_5.STL" />
+        <mesh filename="package://hcr3a/meshes/visual/Link_5.STL" />
       </geometry>
       <material name="">
@@ -147,5 +147,5 @@
       <geometry>
         <mesh
-          filename="file://$(find hcr3a)/meshes/visual/Link_5.STL" />
+          filename="package://hcr3a/meshes/visual/Link_5.STL" />
       </geometry>
     </collision>
@@ -162,5 +162,5 @@
       <origin xyz="0 0 0" rpy="0 0 0" />
       <geometry>
-        <mesh filename="file://$(find hcr3a)/meshes/visual/Link_6.STL" />
+        <mesh filename="package://hcr3a/meshes/visual/Link_6.STL" />
       </geometry>
       <material name="">
@@ -171,5 +171,5 @@
       <origin xyz="0 0 0" rpy="0 0 0" />
       <geometry>
-        <mesh filename="file://$(find hcr3a)/meshes/visual/Link_6.STL" />
+        <mesh filename="package://hcr3a/meshes/visual/Link_6.STL" />
       </geometry>
     </collision>
@@ -186,5 +186,5 @@
       <origin xyz="0 0 0" rpy="0 0 0" />
       <geometry>
-        <mesh filename="file://$(find hcr3a)/meshes/visual/Camera_Link.STL" />
+        <mesh filename="package://hcr3a/meshes/visual/Camera_Link.STL" />
       </geometry>
       <material name="">
@@ -195,5 +195,5 @@
       <origin xyz="0 0 0" rpy="0 0 0" />
       <geometry>
-        <mesh filename="file://$(find hcr3a)/meshes/visual/Camera_Link.STL" />
+        <mesh filename="package://hcr3a/meshes/visual/Camera_Link.STL" />
       </geometry>
     </collision>
@@ -210,5 +210,5 @@
       <origin xyz="0 0 0" rpy="0 0 0" />
       <geometry>
-        <mesh filename="file://$(find hcr3a)/meshes/visual/Forcesensor_Link.STL" />
+        <mesh filename="package://hcr3a/meshes/visual/Forcesensor_Link.STL" />
       </geometry>
       <material name="">
@@ -219,5 +219,5 @@
       <origin xyz="0 0 0" rpy="0 0 0" />
       <geometry>
-        <mesh filename="file://$(find hcr3a)/meshes/visual/Forcesensor_Link.STL" />
+        <mesh filename="package://hcr3a/meshes/visual/Forcesensor_Link.STL" />
       </geometry>
     </collision>
@@ -234,5 +234,5 @@
       <origin xyz="0 0 0" rpy="0 0 0" />
       <geometry>
-        <mesh filename="file://$(find hcr3a)/meshes/visual/Effector_Link.STL" />
+        <mesh filename="package://hcr3a/meshes/visual/Effector_Link.STL" />
       </geometry>
       <material name="">
@@ -243,5 +243,5 @@
       <origin xyz="0 0 0" rpy="0 0 0" />
       <geometry>
-        <mesh filename="file://$(find hcr3a)/meshes/visual/Effector_Link.STL" />
+        <mesh filename="package://hcr3a/meshes/visual/Effector_Link.STL" />
       </geometry>
     </collision>
@@ -258,5 +258,5 @@
       <origin xyz="0 0 0" rpy="0 0 0" />
       <geometry>
-        <mesh filename="file://$(find hcr3a)/meshes/visual/Finger1_Link.STL" />
+        <mesh filename="package://hcr3a/meshes/visual/Finger1_Link.STL" />
       </geometry>
       <material name="">
@@ -267,5 +267,5 @@
       <origin xyz="0 0 0" rpy="0 0 0" />
       <geometry>
-        <mesh filename="file://$(find hcr3a)/meshes/visual/Finger1_Link.STL" />
+        <mesh filename="package://hcr3a/meshes/visual/Finger1_Link.STL" />
       </geometry>
     </collision>
@@ -282,5 +282,5 @@
       <origin xyz="0 0 0" rpy="0 0 0" />
       <geometry>
-        <mesh filename="file://$(find hcr3a)/meshes/visual/Finger2_Link.STL" />
+        <mesh filename="package://hcr3a/meshes/visual/Finger2_Link.STL" />
       </geometry>
       <material name="">
@@ -291,5 +291,5 @@
       <origin xyz="0 0 0" rpy="0 0 0" />
       <geometry>
-        <mesh filename="file://$(find hcr3a)/meshes/visual/Finger2_Link.STL" />
+        <mesh filename="package://hcr3a/meshes/visual/Finger2_Link.STL" />
       </geometry>
     </collision>
