Commit message: gz fix

File: ws_ros2_hanwha/src/hcr3a/urdf/hcr3a_gz_gripper.ros2_control.xacro (robot description, xacro)
@@ -23,7 +23,5 @@
         </state_interface>
       </joint>
-      <joint name="${prefix}finger2">
-        <!-- param name="mimic">${prefix}finger1</param>
-        <param name="multiplier">-1</param -->
+      <!-- joint name="${prefix}finger2">
         <command_interface name="position">
           <param name="min">-0.02557</param>
@@ -41,5 +39,5 @@
           <param name="initial_value">0.0</param>
         </state_interface>
-      </joint>
+      </joint -->
     </ros2_control>
   </xacro:macro>
