Commit message: small changes to planing group

File: ws_ros2_hanwha/src/hcr3a/config/hcr3a_macro.srdf.xacro (robot description, xacro)
@@ -18,13 +18,13 @@
       <link name="finger2_Link" />
       <joint name="finger1" />
-      <joint name="finger2" />
+      <passive_joint name="finger2"/>
     </group>
     <group_state group="gripper" name="open">
       <joint name="finger1" value="0"/>
-      <joint name="finger2" value="0"/>
+      <!-- <joint name="finger2" value="0"/> -->
     </group_state>
     <group_state group="gripper" name="close">
       <joint name="finger1" value="0.025"/>
-      <joint name="finger2" value="-0.025"/>
+      <!-- <joint name="finger2" value="-0.025"/> -->
     </group_state>
     <end_effector group="gripper" name="gripper" parent_group="manipulator" parent_link="forcesensor_Link"/>

File: ws_ros2_hanwha/src/hcr3a/urdf/hcr3a_gripper.ros2_control.xacro (robot description, xacro)
@@ -16,5 +16,5 @@
         <command_interface name="position" />
         <state_interface name="position">
-          <param name="initial_value">0.0</param>
+          <param name="initial_value">0.01</param>
           <param name="min">0</param>
           <param name="max">0.0255</param>

File: ws_ros2_hanwha/src/hcr3a/urdf/hcr3a_macro.xacro (robot description, xacro)
@@ -374,5 +374,5 @@
     <child link="${prefix}finger1_Link" />
     <axis xyz="0 -1 0" />
-    <limit lower="-0.1" upper="0.03" effort="150.0" velocity="1000.0" />
+    <limit lower="-0.03" upper="0.1" effort="150.0" velocity="1000.0" />
     <dynamics damping="0" friction="0"/>
   </joint>
@@ -382,5 +382,5 @@
     <child link="${prefix}finger2_Link" />
     <axis xyz="0 -1 0" />
-    <limit lower="-0.03" upper="0.1" effort="150.0" velocity="1000.0" />
+    <limit lower="-0.1" upper="0.03" effort="150.0" velocity="1000.0" />
     <dynamics damping="0" friction="0"/>
     <mimic joint="${prefix}finger1" multiplier="-1" offset="0" />
